File: CM5IO.kicad_pcb (KiCad board)
At the start: 4 copper layers, 160 x 90 mm, 76 parts, among them J10 690-019-298-412, J11 USB_C_Receptacle_USB2.0, J12 USB3_A, J14 JST_SHBM04B-SRSS-TB, J16 Conn_01x22_Female, J2 Conn_02x07_Odd_Even, J22 690-019-298-412, J3 Conn_01x03, J4 Bus_M.2_Socket_M, J5 Conn_01x22_Female, J6 THD-02-R, J7 Micro_SD_Card_Det, J8 THD-20-R, J9 THD-02-R, SW1 Right angle Tact button, U1 TPD4EUSB30, U12 RT9742SNGV, U18 RT9742GGJ5, U2 TPD4EUSB30, U3 MagJack-A70-112-331N126, U5 74LVC1G07SE-7, U6 AP22653W6, U7 ASEK-32.768KHZ-L-R-T, U8 AP3441SHE-7B

Commit message: fix initial board commit
Parts:
- removed BT1: Battery_Cell, CM5IO:BatteryHolder_Keystone_3034_1x20mm
- removed J22: 690-019-298-412, CM5IO:EDAC 690-019-298-412
- removed SW1: Right angle Tact button, Button_Switch_THT:SW_Tactile_SPST_Angled_PTS645Vx58-2LFS
- removed TP3, TP5: TestPoint, TestPoint:TestPoint_Pad_2.0x2.0mm
- removed U18: RT9742GGJ5, Package_TO_SOT_SMD:SOT-23-5
- removed logo1: KiCad-Logo2_5mm_SilkScreen, Symbol:KiCad-Logo2_5mm_SilkScreen
- added C20: 10uF, PCM_JLCPCB:C_0805, F.Cu at (562.4, 313.6)
- added C21: 10uF, PCM_JLCPCB:C_0805, F.Cu at (562.4, 311.8)
- added C22: 100nF, PCM_JLCPCB:C_0402, F.Cu at (559.5, 320.6)
- added C23: WCAP-ASLI_6.3X7.7, Custom Components:WCAP-ASLI_6.3X7.7_DXL_, F.Cu at (656.5, 325.7)
- added C24: 100nF, PCM_JLCPCB:C_0402, F.Cu at (599.0, 234.0)
- added C25: 100nF, PCM_JLCPCB:C_0402, F.Cu at (633.0, 234.0)
- added C26: 100nF, PCM_JLCPCB:C_0402, F.Cu at (539.0, 234.0)
- added C27: 100nF, PCM_JLCPCB:C_0402, F.Cu at (694.0, 234.0)
- added C28: 100nF, PCM_JLCPCB:C_0402, F.Cu at (539.0, 314.0)
- added C29: 100nF, PCM_JLCPCB:C_0402, F.Cu at (694.0, 314.0)
- added C30: 100nF, PCM_JLCPCB:C_0402, F.Cu at (539.0, 344.0)
- added C31: 100nF, PCM_JLCPCB:C_0402, F.Cu at (694.0, 344.0)
- added C32: 10uF, PCM_JLCPCB:C_0402, F.Cu at (615.9, 254.5)
- added C33: 10uF, PCM_JLCPCB:C_0402, F.Cu at (614.9, 254.5)
- added C34: 10uF, PCM_JLCPCB:C_0402, F.Cu at (609.2, 254.5)
- added C35: 10uF, PCM_JLCPCB:C_0402, F.Cu at (608.2, 254.5)
- added C36: 100nF, PCM_JLCPCB:C_0402, F.Cu at (633.6, 253.4)
- added C37: 100nF, PCM_JLCPCB:C_0402, F.Cu at (633.6, 258.7)
- added F1: 4628, Custom Components:FUSE_4628, F.Cu at (672.1, 363.2)
- added J1: 703W-00_53, Custom Components:QUALTEK_703W-00_53, F.Cu at (671.1, 380.2)
- added J13: JST_SHBM04B-SRSS-TB, Connector_JST:JST_SH_BM04B-SRSS-TB_1x04-1MP_P1.00mm_Vertical, F.Cu at (640.2, 325.0)
- added J15: Bus_M.2_Socket_M, CM5IO:M.2 M Key socket, F.Cu at (577.5, 319.7)
- added J17: SSW-114-01-X-S, Custom Components:SAMTEC_SSW-114-01-X-S, F.Cu at (667.0, 284.8)
- added J18: 6130XX11821_61300811821, Custom Components:61300811821, F.Cu at (651.7, 270.2)
- added J19: 6130XX11821_61300811821, Custom Components:61300811821, F.Cu at (674.6, 270.2)
- added J20: 6130XX11821_61300811821, Custom Components:61300811821, F.Cu at (662.9, 306.8)
- added J21: 6130XX11821_61300811821, Custom Components:61300811821, F.Cu at (662.9, 319.5)
- added MK1: ICS-43434, Sensor_Audio:InvenSense_ICS-43434-6_3.5x2.65mm, F.Cu at (596.8, 236.0)
- added MK2: ICS-43434, Sensor_Audio:InvenSense_ICS-43434-6_3.5x2.65mm, F.Cu at (630.8, 236.0)
- added MK3: ICS-43434, Sensor_Audio:InvenSense_ICS-43434-6_3.5x2.65mm, F.Cu at (536.8, 236.0)
- added MK4: ICS-43434, Sensor_Audio:InvenSense_ICS-43434-6_3.5x2.65mm, F.Cu at (691.8, 236.0)
- added MK5: ICS-43434, Sensor_Audio:InvenSense_ICS-43434-6_3.5x2.65mm, F.Cu at (536.8, 316.0)
- added MK6: ICS-43434, Sensor_Audio:InvenSense_ICS-43434-6_3.5x2.65mm, F.Cu at (691.8, 316.0)
- added MK7: ICS-43434, Sensor_Audio:InvenSense_ICS-43434-6_3.5x2.65mm, F.Cu at (536.8, 346.0)
- added MK8: ICS-43434, Sensor_Audio:InvenSense_ICS-43434-6_3.5x2.65mm, F.Cu at (691.8, 346.0)
- added R11: 2.2kΩ, PCM_JLCPCB:R_0402, F.Cu at (556.5, 312.6)
- added R13: 100Ω, PCM_JLCPCB:R_0603, F.Cu at (594.5, 235.2)
- added R18: 100Ω, PCM_JLCPCB:R_0603, F.Cu at (689.5, 315.2)
- added R19: 100Ω, PCM_JLCPCB:R_0603, F.Cu at (689.5, 345.2)
- added R20: 100Ω, PCM_JLCPCB:R_0603, F.Cu at (534.5, 345.2)
- added R21: 2.2kΩ, PCM_JLCPCB:R_0402, F.Cu at (613.1, 259.0)
- added R22: 100kΩ, PCM_JLCPCB:R_0402, F.Cu at (606.4, 259.0)
- added R23: 33Ω, PCM_JLCPCB:R_0402, F.Cu at (633.6, 252.7)
- added R24: 33Ω, PCM_JLCPCB:R_0402, F.Cu at (624.1, 253.9)
- added R25: 33Ω, PCM_JLCPCB:R_0402, F.Cu at (624.1, 251.9)
- added R26: 33Ω, PCM_JLCPCB:R_0402, F.Cu at (624.1, 253.2)
- added R27: 33Ω, PCM_JLCPCB:R_0402, F.Cu at (633.6, 250.7)
- added R28: 33Ω, PCM_JLCPCB:R_0402, F.Cu at (633.6, 256.0)
- added R29: 33Ω, PCM_JLCPCB:R_0402, F.Cu at (624.1, 258.5)
- added R30: 33Ω, PCM_JLCPCB:R_0402, F.Cu at (624.1, 257.2)
- added R31: 33Ω, PCM_JLCPCB:R_0402, F.Cu at (624.1, 259.2)
- added R32: 33Ω, PCM_JLCPCB:R_0402, F.Cu at (633.6, 258.0)
- added U10: AP3441SHE-7B, Package_DFN_QFN:DFN-8-1EP_2x2mm_P0.5mm_EP1.05x1.75mm, F.Cu at (558.6, 312.3)
- added U11: ASEK-32.768KHZ-L-R-T, Crystal:Crystal_SMD_3225-4Pin_3.2x2.5mm, F.Cu at (562.2, 320.7)
- added U13: MAX98357AETE_T, Custom Components:QFN50P300X300X80-17N, F.Cu at (605.5, 255.7)
- added U14: CDCLVC1106PWR, Custom Components:SOP65P640X120-14N, F.Cu at (628.7, 252.0)
- added U15: CDCLVC1106PWR, Custom Components:SOP65P640X120-14N, F.Cu at (628.7, 257.4)
- added U4: RT9742SNGV, Package_TO_SOT_SMD:TSOT-23_HandSoldering, F.Cu at (538.8, 267.5)
- added U9: MagJack-A70-112-331N126, CM5IO:TRJG0926HENL, F.Cu at (541.6, 364.8)
- added Ue1: L9110S, Custom Components:SOIC127P599X172-8N, F.Cu at (656.9, 349.4)
- C1: value 100n -> 10uF; footprint Capacitor_SMD:C_0402_1005Metric -> PCM_JLCPCB:C_1206
- C10, C13: value 100n -> 100nF; footprint Capacitor_SMD:C_0402_1005Metric -> PCM_JLCPCB:C_0402
- C11: value 4.7nF -> 100nF; footprint Capacitor_SMD:C_0402_1005Metric -> PCM_JLCPCB:C_0402
- C12, C18, C19, C9: value 100n -> 10uF; footprint Capacitor_SMD:C_0402_1005Metric -> PCM_JLCPCB:C_0805
- C14, C15, C6, C8: value 10u -> 10uF; footprint Capacitor_SMD:C_0805_2012Metric -> PCM_JLCPCB:C_0805
- C16: value 10u -> 100nF; footprint Capacitor_SMD:C_0805_2012Metric -> PCM_JLCPCB:C_0402
- C17: value 10u -> 4.7nF; footprint Capacitor_SMD:C_0805_2012Metric -> PCM_JLCPCB:C_0402
- C2: value 10u -> 22uF; footprint Capacitor_SMD:C_0805_2012Metric -> PCM_JLCPCB:C_0805
- C3: value 100uF -> WCAP-FTX2_P22.5_CS; footprint Capacitor_Tantalum_SMD:CP_EIA-7343-31_Kemet-D -> Custom Components:WCAP-FTX2_P22.5L26W6H12_CS
- C4, C5: value 10u -> DE1E3RA472MA4BN01F; footprint Capacitor_SMD:C_0805_2012Metric -> Custom Components:CAP_DE1E3RA472MA4BN01F
- C7: value 10u -> 100nF; footprint Capacitor_SMD:C_0805_2012Metric -> PCM_JLCPCB:C_CASE-B-3528-21(mm)
- D1: value LED Red -> LED Green
- D2: value LED Green -> LED Red
- J10: value 690-019-298-412 -> 691210910004; footprint CM5IO:EDAC 690-019-298-412 -> Custom Components:691210910004
- J11: value USB_C_Receptacle_USB2.0 -> 690-019-298-412; footprint Connector_USB:USB_C_Receptacle_GCT_USB4105-xx-A_16P_TopMnt_Horizontal -> CM5IO:EDAC 690-019-298-412
- J14: value JST_SHBM04B-SRSS-TB -> Micro_SD_Card_Det; footprint Connector_JST:JST_SH_BM04B-SRSS-TB_1x04-1MP_P1.00mm_Vertical -> CM5IO:SDCARD_MOLEX_503398-1892
- J16: value Conn_01x22_Female -> SSW-114-01-X-S; footprint CM5IO:Hirose_FH12-22S-0.5SH_1x22-1MP_P0.50mm_Horizontal -> Custom Components:SAMTEC_SSW-114-01-X-S
- J2: value Conn_02x07_Odd_Even -> B2B-PH-K-S; footprint Connector_PinHeader_2.54mm:PinHeader_2x07_P2.54mm_Vertical -> Custom Components:JST_B2B-PH-K-S
- J3: value Conn_01x03 -> B2B-PH-K-S; footprint Connector_PinHeader_2.54mm:PinHeader_1x03_P2.54mm_Vertical -> Custom Components:JST_B2B-PH-K-S
- J4: value Bus_M.2_Socket_M -> VR10S09; footprint CM5IO:M.2 M Key socket -> Custom Components:VR10S09
- J5: value Conn_01x22_Female -> 691101810005; footprint CM5IO:Hirose_FH12-22S-0.5SH_1x22-1MP_P0.50mm_Horizontal -> Custom Components:691101810005
- J6: value THD-02-R -> 691210910006; footprint Connector_PinHeader_2.54mm:PinHeader_2x02_P2.54mm_Vertical -> Custom Components:691210910006
- J7: value Micro_SD_Card_Det -> 691210910006; footprint CM5IO:SDCARD_MOLEX_503398-1892 -> Custom Components:691210910006
- J8: value THD-20-R -> 5055750471; footprint Connector_PinHeader_2.54mm:PinHeader_2x20_P2.54mm_Vertical -> Custom Components:MOLEX_5055750471
- J9: value THD-02-R -> 1726470103; footprint Connector_PinHeader_2.54mm:PinHeader_2x02_P2.54mm_Vertical -> Custom Components:MOLEX_1726470103
- R1: value 1k -> 15K 1%
- R10: value 1k -> 10kΩ; footprint Resistor_SMD:R_0402_1005Metric -> PCM_JLCPCB:R_0402
- R12: value 15K 1% -> 1kΩ; footprint Resistor_SMD:R_0402_1005Metric -> PCM_JLCPCB:R_0402
- R14: value 100K 1% -> 100Ω; footprint Resistor_SMD:R_0402_1005Metric -> PCM_JLCPCB:R_0603
- R15: value 10K 1% -> 100Ω; footprint Resistor_SMD:R_0402_1005Metric -> PCM_JLCPCB:R_0603
- R16: value 2.2K 1% -> 100Ω; footprint Resistor_SMD:R_0402_1005Metric -> PCM_JLCPCB:R_0603
- R17: value 1k -> 100Ω; footprint Resistor_SMD:R_0402_1005Metric -> PCM_JLCPCB:R_0603
- R2, R3: value 470R -> 7.5kΩ; footprint Resistor_SMD:R_0402_1005Metric -> PCM_JLCPCB:R_0402
- R4: value nf -> 1kΩ; footprint Resistor_SMD:R_0805_2012Metric_Pad1.20x1.40mm_HandSolder -> PCM_JLCPCB:R_0402
- R5: value 0R -> 13kΩ; footprint Resistor_SMD:R_0805_2012Metric_Pad1.20x1.40mm_HandSolder -> PCM_JLCPCB:R_0805
- R6: value 2.2K 1% -> 1kΩ; footprint Resistor_SMD:R_0402_1005Metric -> PCM_JLCPCB:R_0402
- R7, R8: value 2.2K 1% -> 470Ω; footprint Resistor_SMD:R_0402_1005Metric -> PCM_JLCPCB:R_0402
- R9: value 2.2K 1% -> 100kΩ; footprint Resistor_SMD:R_0402_1005Metric -> PCM_JLCPCB:R_0402
- TP1: moved to F.Cu
- U1: value TPD4EUSB30 -> UWS-5_10-Q48N-C; footprint Package_SON:USON-10_2.5x1.0mm_P0.5mm -> Custom Components:VREG_UWS-5_10-Q48N-C; moved to B.Cu
- U12: value RT9742SNGV -> MAX98357AETE_T; footprint Package_TO_SOT_SMD:TSOT-23_HandSoldering -> Custom Components:QFN50P300X300X80-17N
- U2: value TPD4EUSB30 -> RCLAMP3354S.TCT; footprint Package_SON:USON-10_2.5x1.0mm_P0.5mm -> Custom Components:SOT-23-5L_SEM
- U3: value MagJack-A70-112-331N126 -> AP22653W6; footprint CM5IO:TRJG0926HENL -> Package_TO_SOT_SMD:SOT-23-6
- U6: value AP22653W6 -> TPD4EUSB30; footprint Package_TO_SOT_SMD:SOT-23-6 -> Package_SON:USON-10_2.5x1.0mm_P0.5mm
- U7: value ASEK-32.768KHZ-L-R-T -> TPD4EUSB30; footprint Crystal:Crystal_SMD_3225-4Pin_3.2x2.5mm -> Package_SON:USON-10_2.5x1.0mm_P0.5mm
- U8: value AP3441SHE-7B -> RT9742GGJ5; footprint Package_DFN_QFN:DFN-8-1EP_2x2mm_P0.5mm_EP1.05x1.75mm -> Package_TO_SOT_SMD:SOT-23-5
- moved J5 604.7 mm to (619.1, 368.7)
- moved J6 602.0 mm to (669.3, 350.3), turned to 0 degrees
- moved J16 585.4 mm to (667.0, 300.1), turned to 0 degrees
- moved J10 580.3 mm to (679.0, 329.4), turned to 90 degrees
- moved R6 580.1 mm to (672.8, 241.8), turned to -90 degrees
- moved D1 570.0 mm to (676.5, 242.4), turned to -90 degrees
- moved U5 565.5 mm to (673.5, 245.4), turned to 180 degrees
- moved D2 564.3 mm to (674.5, 242.4), turned to -90 degrees
- moved C12 555.4 mm to (658.3, 247.1), turned to 0 degrees
- moved J8 539.7 mm to (551.8, 383.7), turned to 0 degrees
- moved C3 538.1 mm to (672.1, 372.2), turned to 180 degrees
- moved C1 535.4 mm to (641.6, 355.6), turned to -90 degrees
- moved R3 524.6 mm to (663.2, 287.2), turned to -90 degrees
- moved R2 524.5 mm to (665.5, 287.2)
- moved C2 516.7 mm to (653.4, 355.2), turned to -90 degrees
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Connections:
- C1 pad 1: Net-(C1-Pad1) -> GND
- C1 pad 2: GND -> /+24v
- C11 pad 1: /PCIe-M2/M2_3v3 -> /CM5_HighSpeed/HDMI_5v
- C11 pad 2: /PCIe-M2/FB -> GND
- C12 pad 1: /+5v -> /CM5_GPIO ( Ethernet, GPIO, SDCARD)/SD_PWR
- C13 pad 1: /CM5_HighSpeed/HDMI_5v -> Net-(C13-Pad1)
- C14 pad 1: /PCIe-M2/M2_3v3 -> /+5v
- C15 pad 1: /PCIe-M2/M2_3v3 -> /+5v
- C16 pad 1: /PCIe-M2/M2_3v3 -> /+5v
- C17 pad 2: GND -> /PCIe-M2/FB
- C18 pad 1: /+5v -> /PCIe-M2/M2_3v3
- C2 pad 1: /+5v -> /+9v
- C3 pad 1: /CM5_HighSpeed/VBUS -> /AC_neutral2
- C3 pad 2: GND -> /AC_line
- C4 pad 1: /+5v -> /AC_neutral2
- C4 pad 2: GND -> /AC_Earth
- C5 pad 1: /CM5_GPIO ( Ethernet, GPIO, SDCARD)/SD_PWR -> /AC_Earth
- C5 pad 2: GND -> /AC_line
- C9 pad 1: /+5v -> /CM5_HighSpeed/VBUS
- D1 pad 2: /+3.3v -> /+3.3v_P
- D2 pad 2: /+3.3v -> /+3.3v_P
- J10 pad 1: /CM5_HighSpeed/HDMI1_D2_P -> /DRV225/S_B2
- J10 pad 2: GND -> /DRV225/S_B1
- J10 pad 3: /CM5_HighSpeed/HDMI1_D2_N -> /DRV225/S_A1
- J10 pad 4: /CM5_HighSpeed/HDMI1_D1_P -> /DRV225/S_A2
- J14 pad 1: /+5v -> /CM5_GPIO ( Ethernet, GPIO, SDCARD)/SD_DAT2
- J14 pad 2: /CM5_GPIO ( Ethernet, GPIO, SDCARD)/PWM -> /CM5_GPIO ( Ethernet, GPIO, SDCARD)/SD_DAT3
- J14 pad 3: GND -> /CM5_GPIO ( Ethernet, GPIO, SDCARD)/SD_CMD
- J14 pad 4: /CM5_GPIO ( Ethernet, GPIO, SDCARD)/TACHO -> /CM5_GPIO ( Ethernet, GPIO, SDCARD)/SD_PWR
- J16 pad 10: GND -> /DRV225/T_M0
- J16 pad 11: /CM5_HighSpeed/DPHY1_D2_N -> /DRV225/T_M1
- J16 pad 12: /CM5_HighSpeed/DPHY1_D2_P -> /DRV225/T_M2
- J16 pad 13: GND -> /T_RST
- J16 pad 14: /CM5_HighSpeed/DPHY1_D3_N -> /T_INT
- J2 pad 1: GND -> /MaxAmplifier/OUTPL
- J2 pad 2: /CM5_GPIO ( Ethernet, GPIO, SDCARD)/nRPIBOOT -> /MaxAmplifier/OUTNL
- J3 pad 1: /CM5_GPIO ( Ethernet, GPIO, SDCARD)/WL_nDis -> /MaxAmplifier/OUTPR
- J3 pad 2: GND -> /MaxAmplifier/OUTNR
- J4 pad 1: GND -> /+24v
- J4 pad 2: /PCIe-M2/M2_3v3 -> GND
- J4 pad 3: GND -> /+9v
- J5 pad 1: GND -> /+24v
- J5 pad 2: /CM5_HighSpeed/DPHY0_D0_N -> GND
- J5 pad 3: /CM5_HighSpeed/DPHY0_D0_P -> /AC_Earth
- J5 pad 4: GND -> /AC_line
- J5 pad 5: /CM5_HighSpeed/DPHY0_D1_N -> /AC_neutral2
- J6 pad 1: /CM5_GPIO ( Ethernet, GPIO, SDCARD)/ID_SC -> Net-(Ue1-OA)
- J6 pad 2: /CM5_HighSpeed/SCL1 -> Net-(Ue1-OB)
- J6 pad 3: /CM5_GPIO ( Ethernet, GPIO, SDCARD)/ID_SD -> unconnected-(J6-Pad3)
- J6 pad 4: /CM5_HighSpeed/SDA1 -> GND
- J7 pad 1: /CM5_GPIO ( Ethernet, GPIO, SDCARD)/SD_DAT2 -> /PWR_BUT
- J7 pad 2: /CM5_GPIO ( Ethernet, GPIO, SDCARD)/SD_DAT3 -> GND
- J7 pad 3: /CM5_GPIO ( Ethernet, GPIO, SDCARD)/SD_CMD -> /+3.3v_T
- J7 pad 4: /CM5_GPIO ( Ethernet, GPIO, SDCARD)/SD_PWR -> /T_AR
- J7 pad 5: /CM5_GPIO ( Ethernet, GPIO, SDCARD)/SD_CLK -> /T_AG
- J7 pad 6: GND -> /T_AB
- J8 pad 1: /+3.3v -> /T_BotSCL
- J8 pad 2: /+5v -> /T_BotSDA
- J8 pad 3: /CM5_GPIO ( Ethernet, GPIO, SDCARD)/GPIO2 -> /D+
- J8 pad 4: /+5v -> /D-
- J9 pad 1: /CM5_GPIO ( Ethernet, GPIO, SDCARD)/TR1_TAP -> GND
- J9 pad 2: /CM5_GPIO ( Ethernet, GPIO, SDCARD)/TR2_TAP -> /+5v
- J9 pad 3: /CM5_GPIO ( Ethernet, GPIO, SDCARD)/TR0_TAP -> /+24v
- L1 pad 1: Net-(U8-LX) -> Net-(U10-LX)
- Module1 pad 100: /CM5_GPIO ( Ethernet, GPIO, SDCARD)/CAM_GPIO1 -> unconnected-(Module1A-CAM_GPIO1-Pad100)
- Module1 pad 101: /CM5_GPIO ( Ethernet, GPIO, SDCARD)/USBOTG -> GND
- Module1 pad 103: /USB2_N -> /D-
- Module1 pad 105: /USB2_P -> /D+
- Module1 pad 20: /CM5_GPIO ( Ethernet, GPIO, SDCARD)/EEPROM_nWP -> GND
- Module1 pad 24: /CM5_GPIO ( Ethernet, GPIO, SDCARD)/GPIO26 -> /SDI3
- Module1 pad 25: /CM5_GPIO ( Ethernet, GPIO, SDCARD)/GPIO21 -> /SDO0
- Module1 pad 26: /CM5_GPIO ( Ethernet, GPIO, SDCARD)/GPIO19 -> /WS
- Module1 pad 27: /CM5_GPIO ( Ethernet, GPIO, SDCARD)/GPIO20 -> /SDI0
- Module1 pad 45: /CM5_GPIO ( Ethernet, GPIO, SDCARD)/GPIO24 -> /SDI2
- Module1 pad 46: /CM5_GPIO ( Ethernet, GPIO, SDCARD)/GPIO22 -> /SDI1
- Module1 pad 49: /CM5_GPIO ( Ethernet, GPIO, SDCARD)/GPIO18 -> /SCLK
- Module1 pad 56: /CM5_GPIO ( Ethernet, GPIO, SDCARD)/GPIO3 -> /T_BotSCL
- Module1 pad 58: /CM5_GPIO ( Ethernet, GPIO, SDCARD)/GPIO2 -> /T_BotSDA
- Module1 pad 78: /CM5_GPIO ( Ethernet, GPIO, SDCARD)/GPIO_VREF -> /+3.3v_P
- Module1 pad 80: /CM5_HighSpeed/SCL0 -> unconnected-(Module1A-SCL0-Pad80)
- Module1 pad 82: /CM5_HighSpeed/SDA0 -> unconnected-(Module1A-SDA0-Pad82)
- Module1 pad 84: /+3.3v -> /+3.3v_P
- Module1 pad 86: /+3.3v -> /+3.3v_P
- Module1 pad 88: /CM5_GPIO ( Ethernet, GPIO, SDCARD)/+1.8v -> Net-(Module1A-+1.8v_(Output)-Pad88)
- Module1 pad 90: /CM5_GPIO ( Ethernet, GPIO, SDCARD)/+1.8v -> Net-(Module1A-+1.8v_(Output)-Pad88)
- Module1 pad 92: /CM5_GPIO ( Ethernet, GPIO, SDCARD)/PWR_BUT -> /PWR_BUT
- Module1 pad 94: /CC1 -> /CM5_GPIO ( Ethernet, GPIO, SDCARD)/CC1
- Module1 pad 96: /CC2 -> /CM5_GPIO ( Ethernet, GPIO, SDCARD)/CC2
- Module1 pad 97: /CM5_GPIO ( Ethernet, GPIO, SDCARD)/CAM_GPIO0 -> unconnected-(Module1A-CAM_GPIO0-Pad97)
- R1 pad 1: Net-(D2-K) -> Net-(U3-ILIM)
- R1 pad 2: Net-(Module1A-LED_nACT) -> GND
- R10 pad 1: Net-(D1-K) -> /PCIe-M2/M2_3v3
- R10 pad 2: Net-(R10-Pad2) -> /PCIe-M2/FB
- R12 pad 1: Net-(U6-ILIM) -> Net-(D3-K)
- R12 pad 2: GND -> Net-(J15-DAS/~{DSS}/~{LED1})
- R14 pad 1: /CM5_HighSpeed/PCIE_PWR_EN -> /SDI0
- R15 pad 1: /PCIe-M2/M2_3v3 -> /SDI1
- R15 pad 2: /PCIe-M2/FB -> GND
- R16 pad 1: /PCIe-M2/FB -> /SDI1
- R17 pad 1: Net-(D3-K) -> /SDI2
- R17 pad 2: Net-(J4-DAS/~{DSS}/~{LED1}) -> GND
- R2 pad 1: Net-(U3-LEDY_K) -> /+3.3v_P
- R2 pad 2: /CM5_GPIO ( Ethernet, GPIO, SDCARD)/ETH_LEDG -> /T_BotSCL
- R3 pad 1: Net-(U3-LEDG_K) -> /T_BotSDA
- R3 pad 2: /CM5_GPIO ( Ethernet, GPIO, SDCARD)/ETH_LEDY -> /+3.3v_P
- R4 pad 1: /CM5_GPIO ( Ethernet, GPIO, SDCARD)/+1.8v -> Net-(D1-K)
- R4 pad 2: /CM5_GPIO ( Ethernet, GPIO, SDCARD)/GPIO_VREF -> Net-(Module1A-LED_nACT)
- R5 pad 1: /+3.3v -> /CM5_GPIO ( Ethernet, GPIO, SDCARD)/SD_PWR_ON
- R5 pad 2: /CM5_GPIO ( Ethernet, GPIO, SDCARD)/GPIO_VREF -> /+3.3v_P
- R6 pad 1: /CM5_GPIO ( Ethernet, GPIO, SDCARD)/GPIO_VREF -> Net-(D2-K)
- R6 pad 2: /CM5_HighSpeed/SDA1 -> Net-(R6-Pad2)
- R7 pad 1: /CM5_GPIO ( Ethernet, GPIO, SDCARD)/GPIO_VREF -> /CM5_GPIO ( Ethernet, GPIO, SDCARD)/ETH_LEDG
- R7 pad 2: /CM5_HighSpeed/SCL1 -> Net-(U9-LEDY_K)
- R8 pad 1: /+3.3v -> /CM5_GPIO ( Ethernet, GPIO, SDCARD)/ETH_LEDY
- R8 pad 2: Net-(J16-Pin_17) -> Net-(U9-LEDG_K)
- R9 pad 1: /+5v -> /CM5_HighSpeed/PCIE_PWR_EN
- U1 pad 1: /CM5_GPIO ( Ethernet, GPIO, SDCARD)/TRD3_P -> /+24v
- U1 pad 2: /CM5_GPIO ( Ethernet, GPIO, SDCARD)/TRD3_N -> GND
- U1 pad 4: /CM5_GPIO ( Ethernet, GPIO, SDCARD)/TRD2_N -> GND
- U1 pad 5: /CM5_GPIO ( Ethernet, GPIO, SDCARD)/TRD2_P -> GND
- U1 pad 6: /CM5_GPIO ( Ethernet, GPIO, SDCARD)/TRD2_P -> unconnected-(U1-TRIM-Pad6)
- U1 pad 7: /CM5_GPIO ( Ethernet, GPIO, SDCARD)/TRD2_N -> /+5v
- U1 pad 8: GND -> /+5v
- U12 pad 1: /+5v -> /SDO0
- U12 pad 2: /CM5_HighSpeed/HDMI_5v -> /+5v
- U2 pad 1: /CM5_GPIO ( Ethernet, GPIO, SDCARD)/TRD1_P -> /T_BotSCL
- U2 pad 2: /CM5_GPIO ( Ethernet, GPIO, SDCARD)/TRD1_N -> GND
- U2 pad 3: GND -> /D-
- U2 pad 4: /CM5_GPIO ( Ethernet, GPIO, SDCARD)/TRD0_N -> /D+
- U2 pad 5: /CM5_GPIO ( Ethernet, GPIO, SDCARD)/TRD0_P -> /T_BotSDA
- U3 pad 1: /CM5_GPIO ( Ethernet, GPIO, SDCARD)/TRD0_P -> /+5v
- U3 pad 2: /CM5_GPIO ( Ethernet, GPIO, SDCARD)/TRD0_N -> GND
- U3 pad 3: /CM5_GPIO ( Ethernet, GPIO, SDCARD)/TRD1_P -> /CM5_HighSpeed/VBUS_EN
- U3 pad 4: Net-(C1-Pad1) -> unconnected-(U3-nFault-Pad4)
- U3 pad 5: Net-(C1-Pad1) -> Net-(U3-ILIM)
- U3 pad 6: /CM5_GPIO ( Ethernet, GPIO, SDCARD)/TRD1_N -> /CM5_HighSpeed/VBUS
- U5 pad 4: Net-(R10-Pad2) -> Net-(R6-Pad2)
- U5 pad 5: /+3.3v -> /+3.3v_P
- U6 pad 1: /+5v -> /CM5_GPIO ( Ethernet, GPIO, SDCARD)/TRD3_P
- U6 pad 2: GND -> /CM5_GPIO ( Ethernet, GPIO, SDCARD)/TRD3_N
- U6 pad 3: /CM5_HighSpeed/VBUS_EN -> GND
- U6 pad 4: unconnected-(U6-nFault-Pad4) -> /CM5_GPIO ( Ethernet, GPIO, SDCARD)/TRD2_N
- U6 pad 5: Net-(U6-ILIM) -> /CM5_GPIO ( Ethernet, GPIO, SDCARD)/TRD2_P
- U6 pad 6: /CM5_HighSpeed/VBUS -> /CM5_GPIO ( Ethernet, GPIO, SDCARD)/TRD2_P
- U7 pad 1: /PCIe-M2/M2_3v3 -> /CM5_GPIO ( Ethernet, GPIO, SDCARD)/TRD1_P
- U7 pad 2: GND -> /CM5_GPIO ( Ethernet, GPIO, SDCARD)/TRD1_N
- U7 pad 3: Net-(J4-SUSCLK) -> GND
- U7 pad 4: /PCIe-M2/M2_3v3 -> /CM5_GPIO ( Ethernet, GPIO, SDCARD)/TRD0_N
- U8 pad 1: /PCIe-M2/FB -> /CM5_GPIO ( Ethernet, GPIO, SDCARD)/SD_PWR
- U8 pad 2: unconnected-(U8-PG-Pad2) -> GND
- U8 pad 3: /+5v -> unconnected-(U8-nFLG-Pad3)
- U8 pad 4: GND -> /CM5_GPIO ( Ethernet, GPIO, SDCARD)/SD_PWR_ON
- U8 pad 5: unconnected-(U8-nc-Pad5) -> /+3.3v_P
Routing:
- net /WS: track 0.00 -> 719.2 mm, vias 0 -> 8
- net /SCLK: track 0.00 -> 712.9 mm, vias 0 -> 10
- net /+3.3v_P: track 0.00 -> 547.2 mm, vias 0 -> 21
- net GND: track 766.8 -> 227.6 mm, vias 477 -> 84
- net /+3.3v: track 324.6 -> 0.00 mm, vias 8 -> 0
- net /SDI1: track 0.00 -> 241.0 mm
- net /SDI2: track 0.00 -> 236.7 mm, vias 0 -> 3
- net /SDI3: track 0.00 -> 220.9 mm, vias 0 -> 5
- net /AC_neutral2: track 0.00 -> 208.4 mm
- net /+5v: track 284.2 -> 463.2 mm, vias 25 -> 13
- net /+24v: track 0.00 -> 163.1 mm, vias 0 -> 1
- net /CM5_GPIO ( Ethernet, GPIO, SDCARD)/VBAT: track 154.8 -> 0.00 mm, vias 2 -> 0
- net /AC_line: track 0.00 -> 139.4 mm
- net /+3.3v_T: track 0.00 -> 136.7 mm
- net /SDI0: track 0.00 -> 125.0 mm, vias 0 -> 2
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- removed copper zone on B.Cu, net /+5v
- removed copper zone on B.Cu, net GND
- removed copper zone on F.Cu, net GND
- removed copper zone on In1.Cu, net GND
- removed copper zone on In2.Cu, net GND
Other:
- board size 160 x 90 mm -> 165 x 165 mm
- board text removed: "Battery CR2032"
- board text removed: "Board thickness : 1.6mm Finished copper weight inners : 24.9um or greater Finished copper weight outers : 35um or greater Board finish : OSP Material type : FR4 Colour of solder resists : Green Colour of silk screens : White Only on the top side Board to : UL94-V0 TG >=130 50R trace width 0.13mm@ 3GHz 90R diff pair width 0.147 spacing 0.253mm @ 2.5GHz 100R diff pair width 0.127 spacing 0.253mm @ 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"
- board text removed: "CAM/DISP 0"
- board text removed: "CAM/DISP 1"
- board text removed: "Compute Module 5"
- board text removed: "Compute Module 5 IO Board"
- board text removed: "Ethernet"
- board text removed: "FAN"
- board text removed: "Fit for 1.8V GPIO"
- board text removed: "Fit for 3.3V GPIO"
- board text removed: "Fit jumper to disable eMMC Boot"
- board text removed: "Fit jumper to disable writing to EEPROM"
- board text removed: "Fit two jumpers for CAM/DISP 1"
- board text removed: "HDMI0"
- board text removed: "HDMI1"
- board text removed: "J16"
- board text removed: "J3 : nBT_Dis GND"
- board text removed: "J5"
- board text removed: "M.2 M Key"
- board text removed: "Made in PRC"
- board text removed: "NB SD card only used for CM5 modules without eMMC"
- board text removed: "PMIC_Enable"
- board text removed: "POE"
- board text removed: "PWR_Button"
- board text removed: "Power Button"
- board text removed: "Power In"
- board text removed: "Raspberry Pi HAT"
- board text removed: "Rev 1"
- board text removed: "SD card"
- board text removed: "SYNC_Out"
- board text removed: "USB Device"
- board text removed: "USB3"
- board text removed: "USB_OTG"
- board text removed: "nWireless_Dis"
