File: CM5IO.kicad_sch (KiCad schematic)
At the start: 12 parts, among them J11 USB_C_Receptacle_USB2.0

Commit message: fix initial board commit
Parts:
- removed C18, C9: 100n, Capacitor_SMD:C_0402_1005Metric, symbol Device:C
- removed J11: USB_C_Receptacle_USB2.0, Connector_USB:USB_C_Receptacle_GCT_USB4105-xx-A_16P_TopMnt_Horizontal, symbol Connector:USB_C_Receptacle_USB2.0_16P
- removed R9: 2.2K 1%, Resistor_SMD:R_0402_1005Metric, symbol Device:R
- added C1: 10uF, PCM_JLCPCB:C_1206, symbol PCM_JLCPCB-Capacitors:1206,10uF
- added C2: 22uF, PCM_JLCPCB:C_0805, symbol PCM_JLCPCB-Capacitors:0805,22uF
- added C3: WCAP-FTX2_P22.5_CS, Custom Components:WCAP-FTX2_P22.5L26W6H12_CS, symbol WCAP-FTX2_P22.5_CS:WCAP-FTX2_P22.5_CS
- added C36, C37: 100nF, PCM_JLCPCB:C_0402, symbol PCM_JLCPCB-Capacitors:0402,100nF
- added C4, C5: DE1E3RA472MA4BN01F, Custom Components:CAP_DE1E3RA472MA4BN01F, symbol DE1E3RA472MA4BN01F:DE1E3RA472MA4BN01F
- added F1: 4628, Custom Components:FUSE_4628, symbol 4628:4628
- added J1: 703W-00_53, Custom Components:QUALTEK_703W-00_53, symbol 703W-00_53:703W-00_53
- added J10: 691210910004, Custom Components:691210910004, symbol 691210910004:691210910004
- added J2, J3: B2B-PH-K-S, Custom Components:JST_B2B-PH-K-S, symbol B2B-PH-K-S:B2B-PH-K-S
- added J4: VR10S09, Custom Components:VR10S09, symbol VR10S09:VR10S09
- added J5: 691101810005, Custom Components:691101810005, symbol 691101810005:691101810005
- added J6, J7: 691210910006, Custom Components:691210910006, symbol 691210910006:691210910006
- added J8: 5055750471, Custom Components:MOLEX_5055750471, symbol 5055750471:5055750471
- added J9: 1726470103, Custom Components:MOLEX_1726470103, symbol 1726470103:1726470103
- added R23, R24, R25, R26, R27, R28, R29, R30, R31, R32: 33Ω, PCM_JLCPCB:R_0402, symbol PCM_JLCPCB-Resistors:0402,33Ω
- added U1: UWS-5_10-Q48N-C, Custom Components:VREG_UWS-5_10-Q48N-C, symbol UWS-5_10-Q48N-C:UWS-5_10-Q48N-C
- added U14, U15: CDCLVC1106PWR, Custom Components:SOP65P640X120-14N, symbol CDCLVC1106PWR:CDCLVC1106PWR
- added U2: RCLAMP3354S.TCT, SOT-23-5L_SEM, symbol RCLAMP3354S_TCT:RCLAMP3354S.TCT
- added Ue1: L9110S, Custom Components:SOIC127P599X172-8N, symbol L9110S:L9110S
Connections:
- net +5v: now also J9.2, U1.7 (+SENSE), U1.8 (+VOUT)
- net GND: now also C1.1, C2.2, C36.1, C37.1, J4.2, J5.2, J6.4, J7.2, J8.S1 (SHIELD1), J8.S2 (SHIELD2), J9.1, U1.2 (ON/OFF), U1.3 (-VIN), U1.4 (-VOUT), U1.5 (-SENSE), U14.10 (GND__2), U14.4 (GND), U14.7 (GND__1), U15.10 (GND__2), U15.4 (GND), U15.7 (GND__1), U2.2, Ue1.5 (GND), Ue1.8 (GND)
- new net: R31.1, U15.14 (Y1)
- new net: R27.1, U14.6 (Y4)
- new net: R25.1, U14.11 (Y2)
- new net: R26.1, U14.13 (Y3)
- new net: R32.1, U15.3 (Y0)
- new net: R28.1, U15.6 (Y4)
- new net: R24.1, U14.14 (Y1)
- new net: R23.1, U14.3 (Y0)
- new net: R30.1, U15.11 (Y2)
- new net: R29.1, U15.13 (Y3)
- new net: J6.1, Ue1.1 (OA)
- new net: J6.2, Ue1.4 (OB)
- new net +24v: C1.2, J4.1, J5.1, J9.3, U1.1 (+VIN)
- new net +3.3v_P: C36.2, C37.2, U14.12 (VDD__2), U14.2 (1G), U14.5 (VDD), U14.8 (VDD__1), U15.12 (VDD__2), U15.2 (1G), U15.5 (VDD), U15.8 (VDD__1)
- new net +3.3v_T: J6.6, J7.3
- new net +9v: C2.1, J4.3, Ue1.2 (VCC), Ue1.3 (VCC)
- new net AC_Earth: C4.2, C5.1, J1.2 (EARTH), J5.3
- new net AC_line: C3.2, C5.2, J1.3 (LINE), J5.4
- new net AC_neutral1: F1.1, J1.1 (NEUTRAL)
- new net AC_neutral2: C3.1, C4.1, F1.2, J5.5
- new net D+: J8.3, U2.4
- new net D-: J8.4, U2.3
- new net DRV225/S_A1: J10.3
- new net DRV225/S_A2: J10.4
- new net DRV225/S_B1: J10.2
- new net DRV225/S_B2: J10.1
- new net MaxAmplifier/OUTNL: J2.2
- new net MaxAmplifier/OUTNR: J3.2
- new net MaxAmplifier/OUTPL: J2.1
- new net MaxAmplifier/OUTPR: J3.1
- new net PWR_BUT: J7.1
- new net SCLK: R28.2, R29.2, R30.2, R31.2, R32.2, U15.1 (CLKIN)
- new net T_A0: J6.5
- new net T_AB: J7.6
- new net T_AG: J7.5
- new net T_AR: J7.4
- new net T_BotSCL: J8.1, U2.1
- new net T_BotSDA: J8.2, U2.5
- new net T_IA: Ue1.6 (IA)
- new net T_IB: Ue1.7 (IB)
- new net WS: R23.2, R24.2, R25.2, R26.2, R27.2, U14.1 (CLKIN)
- no-connect marks 2 -> 4
Other:
- added sheet BNO086 (BNO086.kicad_sch)
- added sheet DRV225 (DRV225.kicad_sch)
- added sheet MaxAmplifier (MaxAmplifier.kicad_sch)
- added sheet StereoMic (StereoMic.kicad_sch)
- added sheet StereoMic1 (StereoMic.kicad_sch)
- added sheet StereoMic2 (StereoMic.kicad_sch)
- added sheet StereoMic3 (StereoMic.kicad_sch)
- added sheet Teensy_4.0_Harness (Teensy_4.0_Harness.kicad_sch)
- sheet CM5_GPIO ( Ethernet, GPIO, SDCARD) ports: added +3.3v_P, PWR_BUT, SCL1, SCLK, SDA1, SDI0, SDI1, SDI2, SDI3, SDO0, WS; removed +3.3v, CAM_GPIO0, CAM_GPIO1, CC1, CC2, GPIO_VREF, ID_SC, ID_SD, SCL0, SDA0, USBOTG
- sheet CM5_HighSpeed ports: added none; removed +3.3v, CAM_GPIO0, CAM_GPIO1, GPIO_VREF, ID_SC, ID_SD, SCL0, SDA0, USBOTG_ID
- note added: "Connectors ------- Ethernet SDCARD I2C Fan"
- note added: "Connectors ------- HDMI 0 I2C I2S"
- note added: "Roles ----- Base Motor Base BNO086 Data"
- note removed: "Connectors ------- Ethernet SDCARD 40way RPI Jumpers Fan Battery"
- note removed: "Connectors ------- HDMI 0 HDMI 1 CSI/DSI 0 CSI/DSI 1"
- note removed: "Discharge Resistor Needed by some Type C PSUs"
- note removed: "TypeC Power connector"
- company: Copyright © 2024 Raspberry Pi Ltd. -> Maxwell Stoughton
- title: Compute Module 5 IO Board - Top Level -> N3-Base
- moved on the sheet: H1, H2, H3, H4, H5, H6, H7, H8
