File: PCIe-M2.kicad_sch (KiCad schematic)
At the start: 24 parts, among them J4 Bus_M.2_Socket_M, M1 M.2 Screw, M2 M.2 Solder Nut, M3 M.2 Solder Nut, M4 M.2 Solder Nut, M5 M.2 Solder Nut, U7 ASEK-32.768KHZ-L-R-T, U8 AP3441SHE-7B

Commit message: fix initial board commit
Parts:
- removed C10, C19: 100n, Capacitor_SMD:C_0402_1005Metric, symbol Device:C
- removed C11: 4.7nF, Capacitor_SMD:C_0402_1005Metric, symbol Device:C
- removed C14, C15, C16, C17, C4, C6: 10u, Capacitor_SMD:C_0805_2012Metric, symbol Device:C
- removed R14: 100K 1%, Resistor_SMD:R_0402_1005Metric, symbol Device:R
- removed R15: 10K 1%, Resistor_SMD:R_0402_1005Metric, symbol Device:R
- removed R16: 2.2K 1%, Resistor_SMD:R_0402_1005Metric, symbol Device:R
- removed R17: 1k, Resistor_SMD:R_0402_1005Metric, symbol Device:R
- added C14, C15, C18, C19, C20, C21: 10uF, PCM_JLCPCB:C_0805, symbol PCM_JLCPCB-Capacitors:0805,10uF
- added C16, C22: 100nF, PCM_JLCPCB:C_0402, symbol PCM_JLCPCB-Capacitors:0402,100nF
- added C17: 4.7nF, PCM_JLCPCB:C_0402, symbol PCM_JLCPCB-Capacitors:0402,4.7nF
- added R10: 10kΩ, PCM_JLCPCB:R_0402, symbol PCM_JLCPCB-Resistors:0402,10kΩ
- added R11: 2.2kΩ, PCM_JLCPCB:R_0402, symbol PCM_JLCPCB-Resistors:0402,2.2kΩ
- added R12: 1kΩ, PCM_JLCPCB:R_0402, symbol PCM_JLCPCB-Resistors:0402,1kΩ
- added R9: 100kΩ, PCM_JLCPCB:R_0402, symbol PCM_JLCPCB-Resistors:0402,100kΩ
- renumbered J4 to J15, M5 to M1, M4 to M2, M2 to M4, M1 to M5, U8 to U10, U7 to U11
Connections:
- net +5v: now also C14.1, C15.1, C16.1
- net FB: now also C17.2, R10.2, R11.1
- net GND: now also C14.2, C15.2, C16.2, C18.2, C19.2, C20.2, C21.2, C22.2, R11.2, R9.2
- net M2_3v3: now also C17.1, C18.1, C19.1, C20.1, C21.1, C22.1, R10.1
- net PCIE_PWR_EN: now also R9.1
- net at D3.1 (K), TP1.1: now also R12.1
- net at J15.10 (DAS/~{DSS}/~{LED1}): now also R12.2
Other:
- company: Copyright © 2024 Raspberry Pi Ltd. -> Maxwell Stoughton
- title: Compute Module 5 IO Board - M2 Socket -> PCIE Highspeed Data
